File: pcbs/chips-34.kicad_pcb (KiCad board)
At the start: 2 copper layers, 95.2 x 88.1 mm, 27 parts

Commit message: update kicad files to new version .3
Parts:
- removed B3, B4: , E73:SW_TACT_ALPS_SKQGABE010
- removed the G*** at (238.8, 172.7)
- removed the G*** at (185.4, 140.1)
- removed the G*** at (227.3, 140.1)
- removed the G*** at (225.1, 172.7)
- added ?: , , F.Cu at (12.7, -68.6)
- added ?: , , F.Cu at (70.0, -58.0)
- added ?: , , F.Cu at (25.8, 2.15)
- added G***: LOGO, LOGO, F.Cu at (0.31, 17.8)
- added G***: LOGO, LOGO, F.Cu at (39.1, -9.35)
- added G***: LOGO, LOGO, B.Cu at (39.1, -9.35)
- added JST1: , JST_PH_S2B-PH-K_02x2.00mm_Angled, F.Cu at (13.2, 4.17)
- added JST2: , JST_PH_S2B-PH-K_02x2.00mm_Angled, F.Cu at (16.0, 1.77)
- added REF**: VIA-0.6mm, VIA-0.6mm, F.Cu at (82.9, -8.52)
- added REF**: VIA-0.6mm, VIA-0.6mm, F.Cu at (87.7, 10.5)
- added REF**: VIA-0.6mm, VIA-0.6mm, F.Cu at (51.3, -32.6)
- added REF**: VIA-0.6mm, VIA-0.6mm, F.Cu at (44.9, -36.1)
- added REF**: VIA-0.6mm, VIA-0.6mm, F.Cu at (13.3, -33.6)
- added REF**: VIA-0.6mm, VIA-0.6mm, F.Cu at (70.3, -29.8)
- added REF**: VIA-0.6mm, VIA-0.6mm, F.Cu at (82.9, -27.6)
- added REF**: VIA-0.6mm, VIA-0.6mm, F.Cu at (25.9, -31.4)
- added REF**: VIA-0.6mm, VIA-0.6mm, F.Cu at (13.0, 17.0)
- added REF**: VIA-0.6mm, VIA-0.6mm, F.Cu at (51.3, -13.6)
- added REF**: VIA-0.6mm, VIA-0.6mm, F.Cu at (15.0, 17.0)
- added REF**: VIA-0.6mm, VIA-0.6mm, F.Cu at (70.3, -48.8)
- added REF**: VIA-0.6mm, VIA-0.6mm, F.Cu at (63.9, -11.4)
- added REF**: VIA-0.6mm, VIA-0.6mm, F.Cu at (38.0, 3.21)
- added REF**: VIA-0.6mm, VIA-0.6mm, F.Cu at (63.9, -30.4)
- added REF**: VIA-0.6mm, VIA-0.6mm, F.Cu at (-5.70, -5.00)
- added REF**: VIA-0.6mm, VIA-0.6mm, F.Cu at (-5.70, -43.1)
- added REF**: VIA-0.6mm, VIA-0.6mm, F.Cu at (32.3, -38.3)
- added REF**: VIA-0.6mm, VIA-0.6mm, F.Cu at (82.9, -46.6)
- added REF**: VIA-0.6mm, VIA-0.6mm, F.Cu at (51.3, -51.7)
- added REF**: VIA-0.6mm, VIA-0.6mm, F.Cu at (32.3, -19.3)
- added REF**: VIA-0.6mm, VIA-0.6mm, F.Cu at (13.3, -14.5)
- added REF**: VIA-0.6mm, VIA-0.6mm, F.Cu at (13.3, -52.6)
- added REF**: VIA-0.6mm, VIA-0.6mm, F.Cu at (25.9, -12.3)
- added REF**: VIA-0.6mm, VIA-0.6mm, F.Cu at (68.6, 10.5)
- added REF**: VIA-0.6mm, VIA-0.6mm, F.Cu at (75.1, 8.34)
- added REF**: VIA-0.6mm, VIA-0.6mm, F.Cu at (6.90, -21.9)
- added REF**: VIA-0.6mm, VIA-0.6mm, F.Cu at (32.3, -57.4)
- added REF**: VIA-0.6mm, VIA-0.6mm, F.Cu at (6.90, -2.80)
- added REF**: VIA-0.6mm, VIA-0.6mm, F.Cu at (70.3, -10.7)
- added REF**: VIA-0.6mm, VIA-0.6mm, F.Cu at (56.0, 8.34)
- added REF**: VIA-0.6mm, VIA-0.6mm, F.Cu at (25.9, -50.4)
- added REF**: VIA-0.6mm, VIA-0.6mm, F.Cu at (44.9, -55.2)
- added REF**: VIA-0.6mm, VIA-0.6mm, F.Cu at (44.9, -17.1)
- added REF**: VIA-0.6mm, VIA-0.6mm, F.Cu at (6.90, -40.9)
- added REF**: VIA-0.6mm, VIA-0.6mm, F.Cu at (63.9, -49.5)
- added REF**: VIA-0.6mm, VIA-0.6mm, F.Cu at (-5.70, -24.1)
- added REF**: VIA-0.6mm, VIA-0.6mm, F.Cu at (38.0, -5.79)
- added T1, T2: , E73:SPDT_C128955, F.Cu at (14.0, 21.0)
- added TRRS2: TRRS-PJ-320A-dual, TRRS-PJ-320A-dual, F.Cu at (-3.60, -61.8)
- moved TRRS1 261.7 mm to (85.3, -56.4), turned to -90 degrees
- moved B1 242.6 mm to (38.0, -1.29), turned to 180 degrees
- moved B2 242.6 mm to (38.0, -1.29), turned to 180 degrees
- moved S7 231.7 mm to (38.0, -14.3)
- moved S8 231.7 mm to (38.0, -33.3)
- moved S9 231.7 mm to (38.0, -52.4)
- moved S1 229.8 mm to (0.00, 0.00)
- moved S2 229.8 mm to (0.00, -19.1)
- moved S3 229.8 mm to (0.00, -38.1)
- moved S4 229.8 mm to (19.0, -9.53)
- moved S5 229.8 mm to (19.0, -28.6)
- moved S6 229.8 mm to (19.0, -47.6)
- moved S10 229.2 mm to (57.0, -8.57)
- moved S11 229.2 mm to (57.0, -27.6)
- moved S12 229.2 mm to (57.0, -46.7)
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Connections:
- net thumb_stretch renamed thumb_squeeze
- MCU1 pad 11: thumb_resting -> matrix_inner_bottom
- MCU1 pad 13: P9 -> thumb_resting
- MCU1 pad 14: matrix_inner_bottom -> matrix_inner_home
- MCU1 pad 15: matrix_inner_home -> matrix_index_bottom
- MCU1 pad 16: matrix_index_bottom -> matrix_index_top
- MCU1 pad 17: matrix_middle_bottom -> matrix_middle_home
- MCU1 pad 18: matrix_middle_top -> matrix_ring_bottom
- MCU1 pad 19: matrix_ring_bottom -> matrix_ring_top
- MCU1 pad 20: matrix_pinky_bottom -> matrix_pinky_home
- MCU1 pad 23: matrix_pinky_home -> matrix_pinky_top
- MCU1 pad 24: matrix_pinky_top -> P1
- MCU1 pad 5: matrix_ring_top -> matrix_pinky_bottom
- MCU1 pad 7: matrix_middle_home -> matrix_middle_top
- MCU1 pad 8: matrix_index_top -> matrix_middle_bottom
- TRRS1 pad 1: VCC -> GND
- TRRS1 pad 2: P2 -> GND
- TRRS1 pad 3: P3 -> P1
- TRRS1 pad 4: GND -> VCC
Routing:
- net GND: track 603.4 -> 903.8 mm
- net P1: track 0.00 -> 210.5 mm
- net VCC: track 46.8 -> 234.4 mm
- net P9: track 91.1 -> 0.00 mm
- net RST: track 126.9 -> 38.1 mm
- net thumb_resting: track 84.6 -> 41.9 mm
- net thumb_squeeze: track 60.8 -> 21.3 mm
- net matrix_pinky_top: track 71.7 -> 106.9 mm
- net matrix_pinky_home: track 53.3 -> 83.9 mm
- net BAT: track 0.00 -> 21.6 mm
- net matrix_inner_bottom: track 77.9 -> 56.5 mm
- net matrix_pinky_bottom: track 31.1 -> 50.9 mm
- net matrix_ring_bottom: track 43.4 -> 62.5 mm
- net matrix_index_bottom: track 64.2 -> 45.3 mm
- net matrix_ring_home: track 62.1 -> 79.5 mm
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Other:
- board size 95.2 x 88.1 mm -> 99.8 x 84.8 mm
- board text added: "by xandeire"
- board text added: "chips34"
- board text added: "v0.3"
- board text removed: "-v0.1-"
- board text removed: "CHEAP AS"
- board text removed: "COLEMAK"
- board text removed: "IRE"
- board text removed: "QUERTY"
- board text removed: "RESET"
- board text removed: "Xander"
